Commit message: fixed kinova

File: gen3/kortex_dual/config/kinova.urdf.xacro (robot description, xacro)
@@ -66,10 +66,10 @@
       <origin rpy="0 0 0" xyz="0 0 0.17"/>
       <geometry>
-	<mesh filename="package://ur_dual_bringup/meshes/nosac.stl" scale="0.001 0.001 0.001"/>
+	<mesh filename="package://kortex_dual/meshes/nosac.stl" scale="0.001 0.001 0.001"/>
       </geometry>
     </visual>
     <collision>
       <geometry>
-	<mesh filename="package://ur_dual_bringup/meshes/nosac.stl" scale="0.001 0.001 0.001"/>
+	<mesh filename="package://kortex_dual/meshes/nosac.stl" scale="0.001 0.001 0.001"/>
       </geometry>
     </collision>

File: gen3/kortex_dual/urdf/kinova.urdf.xacro (robot description, xacro)
@@ -40,5 +40,4 @@
   <!-- create link fixed to the "world" -->
   <link name="world" />
-  <link name="world" />
   <link name="ground_plane">
     <visual>
@@ -67,10 +66,10 @@
       <origin rpy="0 0 0" xyz="0 0 0.17"/>
       <geometry>
-	<mesh filename="package://ur_dual_bringup/meshes/nosac.stl" scale="0.001 0.001 0.001"/>
+	<mesh filename="package://kortex_dual/meshes/nosac.stl" scale="0.001 0.001 0.001"/>
       </geometry>
     </visual>
     <collision>
       <geometry>
-	<mesh filename="package://ur_dual_bringup/meshes/nosac.stl" scale="0.001 0.001 0.001"/>
+	<mesh filename="package://kortex_dual/meshes/nosac.stl" scale="0.001 0.001 0.001"/>
       </geometry>
     </collision>
@@ -82,5 +81,5 @@
   </joint>
   <xacro:load_robot
-    parent="world"
+    parent="kinova_carrier"
     arm="$(arg arm)"
     gripper="$(arg gripper)"
@@ -105,5 +104,5 @@
     initial_positions="${xacro.load_yaml(initial_positions_file)}"
     moveit_active="$(arg moveit_active)">
-    <origin xyz="0 0 0" rpy="0 0 0" />  <!-- position robot in the world -->
+    <origin xyz="0 0 0.18" rpy="0 -0.785 0" />  <!-- position robot in the world -->
   </xacro:load_robot>
 </robot>
