Commit message: changed some references to ur_simulation_gz

File: ur5/dual_description/urdf/dual.urdf.xacro (robot description, xacro)
@@ -42,5 +42,5 @@
   <!-- import main macro -->
   <xacro:include filename="$(find ur_description)/urdf/ur_macro.xacro"/>
-  <xacro:include filename="$(find ur_simulation_gz)/urdf/ur_gz.ros2_control.xacro" />
+  <xacro:include filename="$(find ur_dual_bringup)/urdf/ur_gz.ros2_control.xacro" />
   <!-- possible 'ur_type' values: ur3, ur3e, ur5, ur5e, ur7e, ur10, ur10e, ur12e, ur16e, ur8long, ur15, ur18, ur20, ur30 -->
   <!-- the default value should raise an error in case this was called without defining the type -->
@@ -86,10 +86,10 @@
       <origin rpy="0 0 0" xyz="0 0 0.17"/>
       <geometry>
-	<mesh filename="package://ur_simulation_gz/meshes/nosac.stl" scale="0.001 0.001 0.001"/>
+	<mesh filename="package://ur_dual_bringup/meshes/nosac.stl" scale="0.001 0.001 0.001"/>
       </geometry>
     </visual>
     <collision>
       <geometry>
-	<mesh filename="package://ur_simulation_gz/meshes/nosac.stl" scale="0.001 0.001 0.001"/>
+	<mesh filename="package://ur_dual_bringup/meshes/nosac.stl" scale="0.001 0.001 0.001"/>
       </geometry>
     </collision>

File: ur5/dual_moveit_config/srdf/dual.srdf.xacro (robot description, xacro)
@@ -5,5 +5,5 @@
   <xacro:arg name="prefix" default="ur_"/>
   <xacro:include filename="$(find dual_moveit_config)/srdf/gen3.srdf.xacro"/>
-  <xacro:include filename="$(find ur_simulation_gz)/srdf/ur_macro.srdf.xacro"/>
+  <xacro:include filename="$(find ur_dual_bringup)/srdf/ur_macro.srdf.xacro"/>
   <xacro:ur_srdf prefix="$(arg prefix)"/>
   <xacro:kinova_srdf/>

File: ur5/ur_dual_bringup/srdf/ur.srdf.xacro (robot description, xacro)
@@ -4,5 +4,5 @@
   <xacro:arg name="name" default="ur"/>
   <xacro:arg name="prefix" default="ur_"/>
-  <xacro:include filename="$(find ur_simulation_gz)/srdf/ur_macro.srdf.xacro"/>
+  <xacro:include filename="$(find ur_dual_bringup)/srdf/ur_macro.srdf.xacro"/>
   <xacro:ur_srdf prefix="$(arg prefix)"/>
 </robot>

File: ur5/ur_dual_bringup/urdf/ur_gz.urdf.xacro (robot description, xacro)
@@ -5,5 +5,5 @@
   <!-- import main macro -->
   <xacro:include filename="$(find ur_description)/urdf/ur_macro.xacro"/>
-  <xacro:include filename="$(find ur_simulation_gz)/urdf/ur_gz.ros2_control.xacro" />
+  <xacro:include filename="$(find ur_dual_bringup)/urdf/ur_gz.ros2_control.xacro" />
   <!-- possible 'ur_type' values: ur3, ur3e, ur5, ur5e, ur7e, ur10, ur10e, ur12e, ur16e, ur8long, ur15, ur18, ur20, ur30 -->
   <!-- the default value should raise an error in case this was called without defining the type -->
@@ -49,10 +49,10 @@
       <origin rpy="0 0 0" xyz="0 0 0.17"/>
       <geometry>
-	<mesh filename="package://ur_simulation_gz/meshes/nosac.stl" scale="0.001 0.001 0.001"/>
+	<mesh filename="package://ur_dual_bringup/meshes/nosac.stl" scale="0.001 0.001 0.001"/>
       </geometry>
     </visual>
     <collision>
       <geometry>
-	<mesh filename="package://ur_simulation_gz/meshes/nosac.stl" scale="0.001 0.001 0.001"/>
+	<mesh filename="package://ur_dual_bringup/meshes/nosac.stl" scale="0.001 0.001 0.001"/>
       </geometry>
     </collision>

Commit message: changes

File: ur5/dual_description/urdf/dual.urdf.xacro (robot description, xacro)
@@ -82,5 +82,5 @@
     <child link="ground_plane"/>
   </joint>
-  <link name="carrier">
+  <link name="ur_carrier">
     <visual>
       <origin rpy="0 0 0" xyz="0 0 0.17"/>
@@ -95,11 +95,29 @@
     </collision>
   </link>
-  <joint name="carrier_joint" type="fixed">
-    <origin xyz="1.2 0 -0.01" rpy="0 0 0"/>
+  <joint name="ur_carrier_joint" type="fixed">
+    <origin xyz="-0.1 0 -0.01" rpy="0 0 0"/>
     <parent link="ground_plane"/>
-    <child link="carrier"/>
+    <child link="ur_carrier"/>
+  </joint>
+  <link name="kinova_carrier">
+    <visual>
+      <origin rpy="0 0 0" xyz="0 0 0.17"/>
+      <geometry>
+	<mesh filename="package://ur_dual_bringup/meshes/nosac.stl" scale="0.001 0.001 0.001"/>
+      </geometry>
+    </visual>
+    <collision>
+      <geometry>
+	<mesh filename="package://ur_dual_bringup/meshes/nosac.stl" scale="0.001 0.001 0.001"/>
+      </geometry>
+    </collision>
+  </link>
+  <joint name="kinova_carrier_joint" type="fixed">
+    <origin xyz="0.1 0 -0.01" rpy="0 0 3.14"/>
+    <parent link="ground_plane"/>
+    <child link="kinova_carrier"/>
   </joint>
   <xacro:load_robot
-    parent="world"
+    parent="kinova_carrier"
     arm="$(arg arm)"
     gripper="$(arg gripper)"
@@ -124,5 +142,5 @@
     initial_positions="${xacro.load_yaml(initial_positions_file)}"
     moveit_active="$(arg moveit_active)">
-    <origin xyz="0 0 0" rpy="0 0 0" />  <!-- position robot in the world -->
+    <origin xyz="0 0 0.18" rpy="0 -0.7838 0" />  <!-- position robot in the world -->
   </xacro:load_robot>
   <!-- arm -->
@@ -130,5 +148,5 @@
     name="$(arg ur_name)"
     tf_prefix="$(arg ur_prefix)"
-    parent="carrier"
+    parent="ur_carrier"
     joint_limits_parameters_file="$(arg joint_limit_params)"
     kinematics_parameters_file="$(arg kinematics_params)"
@@ -140,5 +158,5 @@
     force_abs_paths="true"
     >
-    <origin xyz="0 0 0.18" rpy="0 -0.785 0" />          <!-- position robot in the world -->
+    <origin xyz="0 0 0.18" rpy="0 -0.7838 0" />          <!-- position robot in the world -->
   </xacro:ur_robot>
   <gazebo reference="world">

Commit message: changed urdf

File: ur5/dual_description/urdf/dual.urdf.xacro (robot description, xacro)
@@ -118,4 +118,10 @@
     <child link="kinova_carrier"/>
   </joint>
+  <link name="tilted_frame"/>
+  <joint name="tilt_joint" type="fixed">
+    <parent link="ur_carrier"/>
+    <child link="tilted_frame"/>
+    <origin xyz="0 0 0.18" rpy="0 -0.7838 0"/>
+  </joint>
   <xacro:load_robot
     parent="kinova_carrier"
@@ -142,5 +148,5 @@
     initial_positions="${xacro.load_yaml(initial_positions_file)}"
     moveit_active="$(arg moveit_active)">
-    <origin xyz="0 0 0.18" rpy="0 -0.7838 0" />  <!-- position robot in the world -->
+    <origin xyz="0 0 0.18" rpy="0 0.7838 3.1416" />  <!-- position robot in the world -->
   </xacro:load_robot>
   <!-- arm -->
@@ -148,5 +154,5 @@
     name="$(arg ur_name)"
     tf_prefix="$(arg ur_prefix)"
-    parent="ur_carrier"
+    parent="tilted_frame"
     joint_limits_parameters_file="$(arg joint_limit_params)"
     kinematics_parameters_file="$(arg kinematics_params)"
@@ -158,5 +164,5 @@
     force_abs_paths="true"
     >
-    <origin xyz="0 0 0.18" rpy="0 -0.7838 0" />          <!-- position robot in the world -->
+    <origin xyz="0 0 0" rpy="0 0 0" />          <!-- position robot in the world -->
   </xacro:ur_robot>
   <gazebo reference="world">

Commit message: changed urdf

File: ur5/dual_description/urdf/dual.urdf.xacro (robot description, xacro)
@@ -164,5 +164,5 @@
     force_abs_paths="true"
     >
-    <origin xyz="0 0 0" rpy="0 0 0" />          <!-- position robot in the world -->
+    <origin xyz="0 0 1.57" rpy="0 0 0" />          <!-- position robot in the world -->
   </xacro:ur_robot>
   <gazebo reference="world">

Commit message: added table

File: ur5/dual_description/urdf/dual.urdf.xacro (robot description, xacro)
@@ -148,5 +148,5 @@
     initial_positions="${xacro.load_yaml(initial_positions_file)}"
     moveit_active="$(arg moveit_active)">
-    <origin xyz="0 0 0.18" rpy="0 0.7838 3.1416" />  <!-- position robot in the world -->
+    <origin xyz="0 0 0" rpy="0 0.7838 3.1416" />  <!-- position robot in the world -->
   </xacro:load_robot>
   <!-- arm -->
@@ -164,5 +164,5 @@
     force_abs_paths="true"
     >
-    <origin xyz="0 0 1.57" rpy="0 0 0" />          <!-- position robot in the world -->
+    <origin xyz="0 0 0" rpy="0 0 1.57" />          <!-- position robot in the world -->
   </xacro:ur_robot>
   <gazebo reference="world">
