Commit message: added kortex control

File: gen3/kortex_dual/urdf/kinova.urdf.xacro (robot description, xacro)
@@ -39,4 +39,5 @@
   <xacro:property name="ros_namespace_prop" value="$(arg ros_namespace)"/>
   <!-- create link fixed to the "world" -->
+  <link name="world" />
   <link name="world" />
   <link name="ground_plane">
@@ -81,5 +82,5 @@
   </joint>
   <xacro:load_robot
-    parent="kinova_carrier"
+    parent="world"
     arm="$(arg arm)"
     gripper="$(arg gripper)"
@@ -104,83 +105,5 @@
     initial_positions="${xacro.load_yaml(initial_positions_file)}"
     moveit_active="$(arg moveit_active)">
-    <origin xyz="0 0 0.18" rpy="0 -0.785 0" />  <!-- position robot in the world -->
+    <origin xyz="0 0 0" rpy="0 0 0" />  <!-- position robot in the world -->
   </xacro:load_robot>
-  <xacro:if value="$(arg sim_gazebo)">
-    <!-- Gazebo plugins -->
-    <gazebo reference="world">
-    </gazebo>
-    <gazebo>
-       <plugin filename="gz_ros2_control-system" name="gz_ros2_control::GazeboSimROS2ControlPlugin">
-        <parameters>$(arg simulation_controllers)</parameters>
-        <controller_manager_node_name>controller_manager</controller_manager_node_name>
-	<ros>
-	  <namespace>kinova</namespace>
-	</ros>
-      </plugin>
-      <plugin filename="gz-sim-sensors-system" name="gz::sim::systems::Sensors">
-        <render_engine>$(arg gazebo_renderer)</render_engine>
-      </plugin>
-    </gazebo>
-    <gazebo reference="camera_color_frame">
-      <sensor name="camera_sensor" type="rgbd_camera">
-        <camera>
-          <horizontal_fov>1.047</horizontal_fov>
-          <image>
-            <width>$(arg camera_width)</width>
-            <height>$(arg camera_height)</height>
-            <format>RGB_INT8</format>
-          </image>
-          <clip>
-            <near>0.1</near>
-            <far>5</far>
-          </clip>
-          <distortion>
-            <k1>0.0</k1>
-            <k2>0.0</k2>
-            <k3>0.0</k3>
-            <p1>0.0</p1>
-            <p2>0.0</p2>
-            <center>0.5 0.5</center>
-          </distortion>
-          <lens>
-            <intrinsics>
-              <fx>554.25469</fx>
-              <fy>554.25469</fy>
-              <cx>320.5</cx>
-              <cy>240.5</cy>
-              <s>0</s>
-            </intrinsics>
-            <!-- These need to match the intrinsics above or
-            Gazebo will default to different default values -->
-            <projection>
-              <p_fx>554.25469</p_fx>
-              <p_fy>554.25469</p_fy>
-              <p_cx>320.5</p_cx>
-              <p_cy>240.5</p_cy>
-              <tx>0</tx>
-              <ty>0</ty>
-            </projection>
-          </lens>
-          <noise>
-            <type>gaussian</type>
-            <mean>0</mean>
-            <stddev>0.00</stddev>
-          </noise>
-          <depth_camera>
-            <clip>
-              <near>0.25</near>
-              <far>5</far>
-            </clip>
-          </depth_camera>
-          <optical_frame_id>color_optical_frame</optical_frame_id>
-        </camera>
-        <gz_frame_id>camera_color_frame</gz_frame_id>
-        <always_on>1</always_on>
-        <update_rate>$(arg camera_fps)</update_rate>
-        <visualize>true</visualize>
-        <topic>wrist_mounted_camera</topic>
-        <enable_metrics>false</enable_metrics>
-      </sensor>
-    </gazebo>
-  </xacro:if>
 </robot>

Commit message: changes

File: gen3/kortex_dual/urdf/kinova.urdf.xacro (robot description, xacro)
@@ -29,8 +29,16 @@
   <xacro:arg name="camera_fps" default="6"/>
   <xacro:arg name="ros_namespace" default=""/>
+  <!-- desk pose in world (default: top of desk at z = 0.89, level) -->
+  <xacro:arg name="desk_x" default="0"/>
+  <xacro:arg name="desk_y" default="0"/>
+  <xacro:arg name="desk_z" default="0.89"/>
+  <xacro:arg name="desk_roll"  default="0"/>
+  <xacro:arg name="desk_pitch" default="0"/>
+  <xacro:arg name="desk_yaw"   default="0"/>
   <xacro:arg name="simulation_controllers" default="$(find kortex_description)/arm/$(arg arm)/$(arg dof)dof/config/ros2_controllers.yaml" />
   <xacro:arg name="moveit_active" default="false"/>
   <!-- import main macro -->
   <xacro:include filename="$(find kortex_description)/robots/kortex_robot.xacro" />
+  <xacro:include filename="$(find rf_lab_setup)/urdf/rf_welding_desk_macro.xacro"/>
   <!-- initial position for simulations (Mock Hardware, Gazebo) -->
   <xacro:arg name="initial_positions_file" default="$(find kortex_description)/config/initial_positions.yaml"/>
@@ -40,26 +48,8 @@
   <!-- create link fixed to the "world" -->
   <link name="world" />
-  <link name="ground_plane">
-    <visual>
-      <origin rpy="0 0 0" xyz="0 0 0"/>
-      <geometry>
-        <box size="5 5 0"/>
-      </geometry>
-      <material name="ground_white">
-        <color rgba="1 1 1 0.5"/>
-      </material>
-    </visual>
-    <collision>
-      <origin rpy="0 0 0" xyz="0 0 0"/>
-      <geometry>
-        <box size="5 5 0"/>
-      </geometry>
-    </collision>
-  </link>
-  <joint name="ground_plane_joint" type="fixed">
-    <origin xyz="0 0 -0.01" rpy="0 0 0"/>
-    <parent link="world"/>
-    <child link="ground_plane"/>
-  </joint>
+  <xacro:rf_welding_desk parent="world">
+    <origin xyz="$(arg desk_x) $(arg desk_y) $(arg desk_z)"
+            rpy="$(arg desk_roll) $(arg desk_pitch) $(arg desk_yaw)"/>
+  </xacro:rf_welding_desk>
   <link name="kinova_carrier">
     <visual>
@@ -76,6 +66,6 @@
   </link>
   <joint name="kinova_carrier_joint" type="fixed">
-    <origin xyz="0.1 0 -0.01" rpy="0 0 3.14"/>
-    <parent link="ground_plane"/>
+    <origin xyz="0.9 0.7 -0.01" rpy="0 0 3.14"/>
+    <parent link="desk_link"/>
     <child link="kinova_carrier"/>
   </joint>
@@ -104,5 +94,5 @@
     initial_positions="${xacro.load_yaml(initial_positions_file)}"
     moveit_active="$(arg moveit_active)">
-    <origin xyz="0 0 0.18" rpy="0 -0.785 0" />  <!-- position robot in the world -->
+    <origin xyz="0 0 0.18" rpy="0 0.7838 3.14" />  <!-- position robot in the world -->
   </xacro:load_robot>
 </robot>
